File: APU.kicad_pcb (KiCad board)
At the start: 2 copper layers, 85 x 65 mm, 45 parts, among them X1 Power, X2 Address, X3 Data, X4 Mode, X5 Control, X6 Clock, X7 Conn_01x10

Commit message: Update
Add F2TTL buffering
Parts:
- added C1: 10u, Capacitor_Tantalum_SMD:CP_EIA-3216-18_Kemet-A_Pad1.58x1.35mm_HandSolder, B.Cu at (101.2, 112.5)
- added C4: 10u, Capacitor_Tantalum_SMD:CP_EIA-3216-18_Kemet-A_Pad1.58x1.35mm_HandSolder, B.Cu at (78.0, 94.8)
- renumbered C8 to C10, C9 to C11, C10 to C12, C11 to C13, C1 to C2, C2 to C3, C3 to C5, C4 to C6, C5 to C7, C6 to C8, C7 to C9
Connections:
- DD1 pad 10: GND -> /F2TTL
- DD1 pad 8: unconnected-(DD1-Pad8) -> Net-(DD2-CLK)
- DD1 pad 9: GND -> /F2TTL
- DD2 pad 23: /F2TTL -> Net-(DD2-CLK)
Routing:
- net Net-(DD2-CLK): track 0.00 -> 50.3 mm, vias 0 -> 1
- net /F2TTL: track 58.9 -> 39.9 mm
- net +12: track 52.9 -> 57.3 mm
- net Net-(DD2-~{END}): track 40.4 -> 44.2 mm
- net +5: track 194.1 -> 196.6 mm
- net /~{FPU_CS}: track 20.2 -> 21.9 mm
- net Net-(DD1-Pad2): track 13.6 -> 12.7 mm
- net /AB0: track 94.3 -> 93.6 mm
- net GND: vias 598 -> 581
Other:
- board text added: "v.1.2 07/08/2026"
- board text removed: "v.1.1 21/05/2026"
