File: APU.kicad_sch (KiCad schematic)
At the start: 42 parts, among them X1 Power, X2 Address, X3 Data, X4 Mode, X5 Control, X6 Clock, X7 Conn_01x10

Commit message: Update
Add F2TTL buffering
Parts:
- added C1, C4: 10u, Capacitor_Tantalum_SMD:CP_EIA-3216-18_Kemet-A_Pad1.58x1.35mm_HandSolder, symbol Device:C_Polarized
- renumbered C8 to C10, C9 to C11, C10 to C12, C11 to C13, C1 to C2, C2 to C3, C3 to C5, C4 to C6, C5 to C7, C6 to C8, C7 to C9
Connections:
- net +12: now also C1.1
- net +5: now also C4.1
- net F2TTL: now also DD1.10, DD1.9; no longer DD2.23 (CLK)
- net GND: now also C1.2, C4.2; no longer DD1.10, DD1.9
- net at DD1.8: now also DD2.23 (CLK)
- no-connect marks 6 -> 5
Other:
- moved on the sheet: C2, C3, C5, C6, DD1C
